Commit message: Add files via upload

File: ee_ur5e_gazebo/urdf/ee_ur5e_table.xacro (robot description, xacro)
@@ -207,3 +207,7 @@
 	    </plugin>
 	</gazebo>
+    <!--Kinect-->
+    <!-- position of kinect has to be changed in common_sensors/urdf/sensors/kinect_properties.urdf.xacro>
+    <xacro:include filename="$(find common_sensors)/urdf/sensors/kinect.urdf.xacro" />
+    <xacro:sensor_kinect parent="d435_link"/-->
 </robot>

File: ee_ur5e_gazebo/urdf/inc/_d435.gazebo.xacro (robot description, xacro)
@@ -25,8 +25,8 @@
       <sensor name="${camera_name}color" type="camera">
         <camera name="${camera_name}">
-          <horizontal_fov>${69.4*deg_to_rad}</horizontal_fov>
+          <horizontal_fov>${85.2*deg_to_rad}</horizontal_fov>  <!--69.4-->
           <image>
-            <width>1920</width>
-            <height>1080</height>
+            <width>1280</width>  <!--1920-->
+            <height>720</height>  <!--1080-->
             <format>RGB_INT8</format>
           </image>
@@ -134,4 +134,6 @@
       	<pointCloudTopicName>depth/points</pointCloudTopicName>
       	<pointCloudCutoff>0.5</pointCloudCutoff>
+	<!--infra_rgb>true</infra_rgb-->
+	<!--alignDepthToColor>true</alignDepthToColor-->
       </plugin>
     </gazebo>

File: ee_ur5e_gazebo/urdf/inc/_d435.urdf.xacro (robot description, xacro)
@@ -15,5 +15,5 @@
     <xacro:property name="d435_cam_depth_to_left_ir_offset" value="0.0"/>
     <xacro:property name="d435_cam_depth_to_right_ir_offset" value="-0.050"/>
-    <xacro:property name="d435_cam_depth_to_color_offset" value="0.015"/>
+    <xacro:property name="d435_cam_depth_to_color_offset" value="0.015"/> <!--0.015-->
     <!-- The following values model the aluminum peripherial case for the
   	D435 camera, with the camera joint represented by the actual
